File: IGN6.kicad_sch (KiCad schematic)
At the start: 24 parts

Commit message: ok
Parts:
- gave numbers to parts that had none: 6
- renumbered R7 to R17, R7 to R18, R7 to R19, R14 to R20, R14 to R21, R14 to R22, R7 to R23, R7 to R24, R7 to R25, R14 to R26, R14 to R27, R14 to R28
Changed lines of the file:
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@@
 (kicad_sch
-	(version 20231120)
+	(version 20250114)
 	(generator "eeschema")
-	(generator_version "8.0")
+	(generator_version "9.0")
 	(paper "A4")
 	(title_block
@@
 		(company "rusEFI.com")
 	)
+	(text "Remove R20-R22, R26-R28, and install Q7-Q12 for use with dumb coils"
+		(exclude_from_sim no)
+		(at 106.68 58.42 0)
+		(effects
+			(font
+				(size 1.27 1.27)
+			)
+			(justify left bottom)
+		)
+	)
 	(junction
 		(at 118.11 64.77)
@@
 		)
 	)
-	(text "Remove R20-R22, R26-R28, and install Q7-Q12 for use with dumb coils"
-		(exclude_from_sim no)
-		(at 106.68 58.42 0)
+	(hierarchical_label "IN5"
+		(shape input)
+		(at 190.5 97.79 0)
 		(effects
 			(font
 				(size 1.27 1.27)
 			)
-			(justify left bottom)
-		)
-	)
-	(hierarchical_label "IN5"
-		(shape input)
-		(at 190.5 97.79 0)
-		(fields_autoplaced yes)
+			(justify left)
+		)
+	)
+	(hierarchical_label "OUT1"
+		(shape output)
+		(at 113.03 64.77 180)
 		(effects
 			(font
 				(size 1.27 1.27)
 			)
-			(justify left)
-		)
-	)
-	(hierarchical_label "OUT1"
+			(justify right)
+		)
+	)
+	(hierarchical_label "OUT3"
 		(shape output)
-		(at 113.03 64.77 180)
-		(fields_autoplaced yes)
+		(at 113.03 120.65 180)
 		(effects
 			(font
@@
 		)
 	)
-	(hierarchical_label "OUT3"
-		(shape output)
-		(at 113.03 120.65 180)
-		(fields_autoplaced yes)
+	(hierarchical_label "IN2"
+		(shape input)
+		(at 143.51 97.79 0)
 		(effects
 			(font
 				(size 1.27 1.27)
 			)
-			(justify right)
-		)
-	)
-	(hierarchical_label "IN2"
+			(justify left)
+		)
+	)
+	(hierarchical_label "IN6"
 		(shape input)
-		(at 143.51 97.79 0)
-		(fields_autoplaced yes)
+		(at 190.5 125.73 0)
 		(effects
 			(font
@@
 		)
 	)
-	(hierarchical_label "IN6"
-		(shape input)
-		(at 190.5 125.73 0)
-		(fields_autoplaced yes)
+	(hierarchical_label "OUT6"
+		(shape output)
+		(at 160.02 120.65 180)
 		(effects
 			(font
 				(size 1.27 1.27)
 			)
-			(justify left)
-		)
-	)
-	(hierarchical_label "OUT6"
+			(justify right)
+		)
+	)
+	(hierarchical_label "OUT5"
 		(shape output)
-		(at 160.02 120.65 180)
-		(fields_autoplaced yes)
+		(at 160.02 92.71 180)
 		(effects
 			(font
@@
 		)
 	)
-	(hierarchical_label "OUT5"
+	(hierarchical_label "OUT2"
 		(shape output)
-		(at 160.02 92.71 180)
-		(fields_autoplaced yes)
+		(at 113.03 92.71 180)
 		(effects
 			(font
@@
 		)
 	)
-	(hierarchical_label "OUT2"
-		(shape output)
-		(at 113.03 92.71 180)
-		(fields_autoplaced yes)
+	(hierarchical_label "IN3"
+		(shape input)
+		(at 143.51 125.73 0)
 		(effects
 			(font
 				(size 1.27 1.27)
 			)
-			(justify right)
-		)
-	)
-	(hierarchical_label "IN3"
+			(justify left)
+		)
+	)
+	(hierarchical_label "IN1"
 		(shape input)
-		(at 143.51 125.73 0)
-		(fields_autoplaced yes)
+		(at 143.51 69.85 0)
 		(effects
 			(font
@@
 		)
 	)
-	(hierarchical_label "IN1"
-		(shape input)
-		(at 143.51 69.85 0)
-		(fields_autoplaced yes)
+	(hierarchical_label "OUT4"
+		(shape output)
+		(at 160.02 64.77 180)
 		(effects
 			(font
 				(size 1.27 1.27)
 			)
-			(justify left)
-		)
-	)
-	(hierarchical_label "OUT4"
-		(shape output)
-		(at 160.02 64.77 180)
-		(fields_autoplaced yes)
-		(effects
-			(font
-				(size 1.27 1.27)
-			)
 			(justify right)
 		)
@@
 		(shape input)
 		(at 190.5 69.85 0)
-		(fields_autoplaced yes)
 		(effects
 			(font
@@
 		(on_board yes)
 		(dnp no)
-		(property "Reference" "Q?"
+		(property "Reference" "Q9"
 			(at 115.7986 124.5616 0)
 			(effects
@@
 		(on_board yes)
 		(dnp no)
-		(property "Reference" "R14"
+		(property "Reference" "R27"
 			(at 177.4796 90.0653 0)
 			(effects
@@
 		(on_board yes)
 		(dnp no)
-		(property "Reference" "R7"
+		(property "Reference" "R17"
 			(at 131.052 67.5018 0)
 			(effects
@@
 		(on_board yes)
 		(dnp no)
-		(property "Reference" "R14"
+		(property "Reference" "R26"
 			(at 177.4796 62.1253 0)
 			(effects
@@
 		(on_board yes)
 		(dnp no)
-		(property "Reference" "R7"
+		(property "Reference" "R25"
 			(at 178.042 123.3818 0)
 			(effects
@@
 		(on_board yes)
 		(dnp no)
-		(property "Reference" "R7"
+		(property "Reference" "R18"
 			(at 131.052 95.4418 0)
 			(effects
@@
 		(on_board yes)
 		(dnp no)
-		(property "Reference" "#PWR?"
+		(property "Reference" "#PWR0101"
 			(at 118.11 142.24 0)
 			(effects
@@
 		(on_board yes)
 		(dnp no)
-		(property "Reference" "R14"
+		(property "Reference" "R20"
 			(at 130.4896 62.1253 0)
 			(effects
@@
 		(on_board yes)
 		(dnp no)
-		(property "Reference" "Q?"
+		(property "Reference" "Q7"
 			(at 115.7986 68.6816 0)
 			(effects
@@
 		(on_board yes)
 		(dnp no)
-		(property "Reference" "#PWR?"
+		(property "Reference" "#PWR0104"
 			(at 165.1 143.51 0)
 			(effects
@@
 		(on_board yes)
 		(dnp no)
-		(property "Reference" "R7"
+		(property "Reference" "R19"
 			(at 131.052 123.3818 0)
 			(effects
@@
 		(on_board yes)
 		(dnp no)
-		(property "Reference" "Q?"
+		(property "Reference" "Q8"
 			(at 115.7986 96.6216 0)
 			(effects
@@
 		(on_board yes)
 		(dnp no)
-		(property "Reference" "#PWR?"
+		(property "Reference" "#PWR099"
 			(at 118.11 86.36 0)
 			(effects
@@
 		(on_board yes)
 		(dnp no)
-		(property "Reference" "Q?"
+		(property "Reference" "Q10"
 			(at 162.7886 68.6816 0)
 			(effects
@@
 		(on_board yes)
 		(dnp no)
-		(property "Reference" "R7"
+		(property "Reference" "R24"
 			(at 178.042 95.4418 0)
 			(effects
@@
 		(on_board yes)
 		(dnp no)
-		(property "Reference" "Q?"
+		(property "Reference" "Q12"
 			(at 162.7886 124.5616 0)
 			(effects
@@
 		(on_board yes)
 		(dnp no)
-		(property "Reference" "R14"
+		(property "Reference" "R28"
 			(at 177.4796 118.0053 0)
 			(effects
@@
 		(on_board yes)
 		(dnp no)
-		(property "Reference" "#PWR?"
+		(property "Reference" "#PWR0102"
 			(at 165.1 87.63 0)
 			(effects
@@
 		(on_board yes)
 		(dnp no)
-		(property "Reference" "R14"
+		(property "Reference" "R21"
 			(at 130.4896 90.0653 0)
 			(effects
@@
 		(on_board yes)
 		(dnp no)
-		(property "Reference" "R7"
+		(property "Reference" "R23"
 			(at 178.042 67.5018 0)
 			(effects
@@
 		(on_board yes)
 		(dnp no)
-		(property "Reference" "#PWR?"
+		(property "Reference" "#PWR0103"
 			(at 165.1 114.3 0)
 			(effects
@@
 		(on_board yes)
 		(dnp no)
-		(property "Reference" "#PWR?"
+		(property "Reference" "#PWR0100"
 			(at 118.11 114.3 0)
 			(effects
@@
 		(on_board yes)
 		(dnp no)
-		(property "Reference" "R14"
+		(property "Reference" "R22"
 			(at 130.4896 118.0053 0)
 			(effects
@@
 		(on_board yes)
 		(dnp no)
-		(property "Reference" "Q?"
+		(property "Reference" "Q11"
 			(at 162.7886 96.6216 0)
 			(effects
