File: LS4.kicad_sch (KiCad schematic)
At the start: 10 parts, among them U7 VNLD5160TR-E, U8 VNLD5160TR-E

Commit message: ok
Parts:
- renumbered D27 to D2, D27 to D3, D27 to D4, D27 to D5, R30 to R10, R30 to R11, R30 to R12, R30 to R13
Changed lines of the file:
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@@
 (kicad_sch
-	(version 20231120)
+	(version 20250114)
 	(generator "eeschema")
-	(generator_version "8.0")
+	(generator_version "9.0")
 	(paper "A4")
 	(title_block
@@
 		(shape input)
 		(at 209.55 85.09 0)
-		(fields_autoplaced yes)
 		(effects
 			(font
@@
 		(shape output)
 		(at 91.44 116.84 180)
-		(fields_autoplaced yes)
 		(effects
 			(font
@@
 		(shape output)
 		(at 91.44 111.76 180)
-		(fields_autoplaced yes)
 		(effects
 			(font
@@
 		(shape output)
 		(at 91.44 90.17 180)
-		(fields_autoplaced yes)
 		(effects
 			(font
@@
 		(shape input)
 		(at 184.15 90.17 0)
-		(fields_autoplaced yes)
 		(effects
 			(font
@@
 		(shape input)
 		(at 209.55 111.76 0)
-		(fields_autoplaced yes)
 		(effects
 			(font
@@
 		(shape output)
 		(at 91.44 85.09 180)
-		(fields_autoplaced yes)
 		(effects
 			(font
@@
 		(shape input)
 		(at 184.15 116.84 0)
-		(fields_autoplaced yes)
 		(effects
 			(font
@@
 		(on_board yes)
 		(dnp no)
-		(property "Reference" "#PWR03"
+		(property "Reference" "#PWR074"
 			(at 106.68 123.19 0)
 			(effects
@@
 		(on_board yes)
 		(dnp no)
-		(property "Reference" "R30"
+		(property "Reference" "R10"
 			(at 194.31 90.17 0)
 			(effects
@@
 		(on_board yes)
 		(dnp no)
-		(property "Reference" "#PWR03"
+		(property "Reference" "#PWR070"
 			(at 106.68 96.52 0)
 			(effects
@@
 		(on_board yes)
 		(dnp no)
-		(property "Reference" "R30"
+		(property "Reference" "R12"
 			(at 194.31 116.84 0)
 			(effects
@@
 		(on_board yes)
 		(dnp no)
-		(property "Reference" "D27"
+		(property "Reference" "D5"
 			(at 104.14 119.38 0)
 			(effects
@@
 		(on_board yes)
 		(dnp no)
-		(property "Reference" "#PWR03"
+		(property "Reference" "#PWR069"
 			(at 106.68 81.28 0)
 			(effects
@@
 		(on_board yes)
 		(dnp no)
-		(property "Reference" "#PWR03"
+		(property "Reference" "#PWR073"
 			(at 106.68 107.95 0)
 			(effects
@@
 		(on_board yes)
 		(dnp no)
-		(property "Reference" "D27"
+		(property "Reference" "D4"
 			(at 104.14 104.14 0)
 			(effects
@@
 		(on_board yes)
 		(dnp no)
-		(property "Reference" "D27"
+		(property "Reference" "D2"
 			(at 104.14 77.47 0)
 			(effects
@@
 		(on_board yes)
 		(dnp no)
-		(property "Reference" "D27"
+		(property "Reference" "D3"
 			(at 104.14 92.71 0)
 			(effects
@@
 		(on_board yes)
 		(dnp no)
-		(property "Reference" "R30"
+		(property "Reference" "R13"
 			(at 168.91 121.92 0)
 			(effects
@@
 		(on_board yes)
 		(dnp no)
-		(property "Reference" "R30"
+		(property "Reference" "R11"
 			(at 168.91 95.25 0)
 			(effects
