File: egt.kicad_sch (KiCad schematic)
At the start: 9 parts, among them U4 MAX31855KASA

Commit message: ok
Parts:
- gave numbers to parts that had none: 5
Changed lines of the file:
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@@
 (kicad_sch
-	(version 20231120)
+	(version 20250114)
 	(generator "eeschema")
-	(generator_version "8.0")
+	(generator_version "9.0")
 	(paper "A4")
 	(title_block
@@
 		(company "rusEFI.com")
 	)
+	(text "NUP2105L is optional, used for protection"
+		(exclude_from_sim no)
+		(at 121.412 114.808 0)
+		(effects
+			(font
+				(size 1.27 1.27)
+			)
+		)
+	)
 	(junction
 		(at 176.53 68.58)
@@
 		)
 	)
-	(text "NUP2105L is optional, used for protection"
-		(exclude_from_sim no)
-		(at 121.412 114.808 0)
+	(hierarchical_label "Vcc"
+		(shape input)
+		(at 201.93 68.58 0)
 		(effects
 			(font
 				(size 1.27 1.27)
 			)
-		)
-	)
-	(hierarchical_label "Vcc"
-		(shape input)
-		(at 201.93 68.58 0)
-		(fields_autoplaced yes)
+			(justify left)
+		)
+	)
+	(hierarchical_label "SPI_SO"
+		(shape output)
+		(at 194.31 90.17 0)
 		(effects
 			(font
@@
 		)
 	)
-	(hierarchical_label "SPI_SO"
-		(shape output)
-		(at 194.31 90.17 0)
-		(fields_autoplaced yes)
+	(hierarchical_label "SPI_SCK"
+		(shape input)
+		(at 194.31 87.63 0)
 		(effects
 			(font
@@
 		)
 	)
-	(hierarchical_label "SPI_SCK"
+	(hierarchical_label "SPI_CS"
 		(shape input)
-		(at 194.31 87.63 0)
-		(fields_autoplaced yes)
+		(at 194.31 95.25 0)
 		(effects
 			(font
@@
 		)
 	)
-	(hierarchical_label "SPI_CS"
+	(hierarchical_label "T+"
 		(shape input)
-		(at 194.31 95.25 0)
-		(fields_autoplaced yes)
+		(at 101.6 87.63 180)
 		(effects
 			(font
 				(size 1.27 1.27)
 			)
-			(justify left)
-		)
-	)
-	(hierarchical_label "T+"
-		(shape input)
-		(at 101.6 87.63 180)
-		(fields_autoplaced yes)
-		(effects
-			(font
-				(size 1.27 1.27)
-			)
 			(justify right)
 		)
@@
 		(shape input)
 		(at 101.6 95.25 180)
-		(fields_autoplaced yes)
 		(effects
 			(font
@@
 		(on_board yes)
 		(dnp no)
-		(property "Reference" "C?"
+		(property "Reference" "C28"
 			(at 138.43 99.695 90)
 			(effects
@@
 		(on_board yes)
 		(dnp no)
-		(property "Reference" "C?"
+		(property "Reference" "C32"
 			(at 191.77 71.755 90)
 			(effects
@@
 		(on_board yes)
 		(dnp no)
-		(property "Reference" "C?"
+		(property "Reference" "C30"
 			(at 153.67 99.695 90)
 			(effects
@@
 		(on_board yes)
 		(dnp no)
-		(property "Reference" "C?"
+		(property "Reference" "C31"
 			(at 179.07 71.755 90)
 			(effects
@@
 		(on_board yes)
 		(dnp no)
-		(property "Reference" "C?"
+		(property "Reference" "C29"
 			(at 144.78 89.535 90)
 			(effects
