File: uaefi.kicad_sch (KiCad schematic)
At the start: 68 parts, among them J1 Conn_02x02_Odd_Even, J1 USB_B_Mini, J1 USB_C, J10 5569-16A2, J11 Conn_02x02_Odd_Even, J12 Conn_02x02_Odd_Even, J13 Conn_02x02_Odd_Even, J14 Conn_02x02_Odd_Even, J15 Conn_02x02_Odd_Even, J16 Conn_02x02_Odd_Even, J17 Conn_01x06, J17 Conn_02x02_Odd_Even, J18 Conn_02x02_Odd_Even, J19 Conn_02x02_Odd_Even, J2 5569-20A2, J20 Conn_02x02_Odd_Even, J21 Conn_02x02_Odd_Even, J22 Conn_02x02_Odd_Even, J24 Conn_02x02_Odd_Even, J3 5569-06A2, J4 5569-08A2, J5 5569-18A2, J5 Conn_01x05_Male, M1 Module-power_12and5V-0.2, M3 Module-knock-0.2, M3 Module-vr-discrete-0.5, M4 Module-vr-max9924-0.1, M5 Module-wbo-0.5, M6 Module:mega-mcu100/0.3, M7 Module-can-0.1, P1 Pad, P2 Pad, P3 Pad, P4 Pad, P5 Pad, P6 Pad, P7 Pad, P8 Pad, U4 JDY-33

Commit message: ok
Parts:
- removed J1, J11, J12, J13, J14, J15, J16, J17, J18, J19, J20, J21, J22, J24: Conn_02x02_Odd_Even, Connector_PinSocket_2.54mm:PinSocket_2x02_P2.54mm_Vertical, symbol Connector_Generic:Conn_02x02_Odd_Even
- removed J10: 5569-16A2, Connector_Molex:Molex_Mini-Fit_Jr_5569-16A2_2x08_P4.20mm_Horizontal, symbol Connector_Generic:Conn_02x08_Top_Bottom
- removed J2: 5569-20A2, Connector_Molex:Molex_Mini-Fit_Jr_5569-20A2_2x10_P4.20mm_Horizontal, symbol Connector_Generic:Conn_02x10_Top_Bottom
- removed J4: 5569-08A2, Connector_Molex:Molex_Mini-Fit_Jr_5569-08A2_2x04_P4.20mm_Horizontal, symbol Connector_Generic:Conn_02x04_Top_Bottom
- removed J5: 5569-18A2, Connector_Molex:Molex_Mini-Fit_Jr_5569-18A2_2x09_P4.20mm_Horizontal, symbol Connector_Generic:Conn_02x09_Top_Bottom
- added D6: SS34, Diode_SMD:D_SMA, symbol Diode:SS34
- added J1: 178780-1_OBD1, kicad6-libraries:178780-1_OBD1, symbol 178780-1:178780-1_OBD1
- added J2: Conn_02x04_Top_Bottom, Connector_Molex:Molex_Micro-Fit_3.0_43045-0812_2x04_P3.00mm_Vertical, symbol Connector_Generic:Conn_02x04_Top_Bottom
- added J4, J5: Conn_02x03_Top_Bottom, Connector_Molex:Molex_Micro-Fit_3.0_43045-0612_2x03_P3.00mm_Vertical, symbol Connector_Generic:Conn_02x03_Top_Bottom
- added P10, P11, P12, P13, P14, P19, P20, P21, P22, P23, P24, P25, P26, P27, P28, P29, P30, P31, P32, P33, P34, P35, P36, P37, P38, P9: Pad, hellen-one-common:PAD-TH, symbol hellen-one-common:Pad
- added Q1: AO3400A, hellen-one-common:SOT-23, symbol Transistor_FET:AO3400A
- added R41, R42, R43, R44, R45, R46, R47, R48, R49, R50, R51, R52, R53, R54, R55, R56, R57, R58, R59, R60, R61, R62, R63, R64, R65, R66, R67, R68, R69, R70, R71, R72: Jumper-Pad-Pad, hellen-one-common:PAD-0805-PAD, symbol hellen-one-common:Jumper-Pad-Pad
- added R73, R74: 0, hellen-one-common:R0603, symbol hellen-one-common:Res
- added U12: BTS6143D, Package_TO_SOT_SMD:TO-252-4, symbol Power_Management:BTS6143D
- J3: value 5569-06A2 -> Conn_02x03_Top_Bottom; footprint Connector_Molex:Molex_Mini-Fit_Jr_5569-06A2_2x03_P4.20mm_Horizontal -> Connector_Molex:Molex_Micro-Fit_3.0_43045-0612_2x03_P3.00mm_Vertical; LCSC C293509 -> (none)
- renumbered C3 to C33, D10 to D1, F6 to F1, F6 to F2, F6 to F3, F6 to F4, J17 to J6, J5 to J7, J1 to J8, J1 to J9, M3 to M2, R30 to R1, R30 to R2, R30 to R3, R38 to R35, R38 to R36, R38 to R37, R41 to R40, R30 to R5, R30 to R6, R3 to R7, R6 to R8, U4 to U5
Connections:
- net +12V_RAW: now also J1.C1, J2.7 (Pin_7); no longer J3.1 (Pin_1)
- net +5VP: now also J3.1 (Pin_1), J3.4 (Pin_4), J4.1 (Pin_1), J4.4 (Pin_4), J5.1 (Pin_1), R43.2, R44.2, R45.2
- net GND: now also J1.A23, J1.A24, J2.8 (Pin_8)
- net GNDA: now also J3.3 (Pin_3), J3.6 (Pin_6), J4.3 (Pin_3), J4.6 (Pin_6), J5.4 (Pin_4), R41.2, R42.2
- net IN_AUX1: now also R50.2
- net IN_AUX2: now also R48.2
- net IN_AUX3: now also R61.2
- net IN_BUTTON1: now also R60.2
- net IN_BUTTON2: now also R54.2
- net IN_BUTTON3: now also R52.2
- net IN_CLT: now also R49.2
- net IN_FLEX: now also J1.C7
- net IN_HALL2: now also R59.2
- net IN_IAT: now also R47.2
- net IN_KNOCK_RAW: now also R53.2
- net IN_MAP: now also R46.2
- net IN_PPS1: now also J3.2 (Pin_2)
- net IN_PPS2: now also J3.5 (Pin_5)
- net IN_TPS1: now also J5.2 (Pin_2), R51.2
- net IN_TPS2: now also J5.5 (Pin_5)
- net OUT_DC1+: now also J5.3 (Pin_3)
- net OUT_DC1-: now also J5.6 (Pin_6)
- net OUT_IGN1: now also J2.1 (Pin_1)
- net OUT_IGN2: now also J2.2 (Pin_2)
- net OUT_IGN3: now also J2.3 (Pin_3)
- net OUT_IGN4: now also J2.4 (Pin_4)
- net OUT_IGN5: now also J2.5 (Pin_5)
- net OUT_INJ1: now also J1.A1
- net OUT_INJ2: now also J1.A3
- net OUT_INJ3: now also J1.A5
- net OUT_INJ4: now also J1.A2
- net OUT_INJ5: now also R71.2
- net OUT_INJ6: now also R66.2
- net OUT_LS1: now also R67.2
- net OUT_LS2: now also R65.2
- net OUT_LS4: now also J1.A7, R73.2
- net VR_DISCRETE+: now also R58.2
- net VR_DISCRETE-: now also R57.2
- net VR_MAX9924+: now also R56.2
- net VR_MAX9924-: now also R55.2
- net WBO_Heater: now also J1.C2; no longer J3.3 (Pin_3)
- net WBO_Ip: now also J1.C4; no longer J3.5 (Pin_5)
- net WBO_Rtrim: now also J1.C5; no longer J3.2 (Pin_2)
- net WBO_Un: now also J1.C6; no longer J3.4 (Pin_4)
- net WBO_Vm: now also J1.C3; no longer J3.6 (Pin_6)
- new net: J1.A16, R67.1
- new net: J1.D20, R43.1
- new net: J1.B11, R58.1
- new net: J1.B13, P24.1 (Pin_1)
- new net: J1.D16, P38.1 (Pin_1)
- new net: J1.C10, P28.1 (Pin_1)
- new net: J1.B8, P23.1 (Pin_1)
- new net: J1.D13, R49.1
- new net: J1.A17, R66.1
- new net: J1.B1, P14.1 (Pin_1)
- new net: J1.B7, P22.1 (Pin_1)
- new net: J1.D12, R50.1
- new net: J1.D8, P35.1 (Pin_1)
- new net: J1.D21, R42.1
- new net: J1.A21, R64.1, R74.2
- new net: J1.D19, R44.1
- new net: J1.D22, R41.1
- new net: J1.D7, P34.1 (Pin_1)
- new net: J1.D15, R47.1
- new net: J1.A22, R74.1
- new net: J1.D2, R54.1
- new net: J1.B3, P19.1 (Pin_1)
- new net: J1.A10, P10.1 (Pin_1)
- new net: J1.A11, R71.1
- new net: J1.A12, R70.1
- new net: J1.A13, R69.1
- new net: J1.A14, P11.1 (Pin_1)
- new net: J1.A15, R68.1
- new net: J1.A18, P12.1 (Pin_1)
- new net: J1.A19, P13.1 (Pin_1)
- new net: J1.A20, R65.1
- new net: J1.A26, R63.1
- new net: J1.A6, P9.1 (Pin_1)
- new net: J1.A8, R73.1
- new net: J1.A9, R72.1
- new net: J1.B10, R59.1
- new net: J1.B12, R57.1
- new net: J1.B14, P25.1 (Pin_1)
- new net: J1.B15, R56.1
- new net: J1.B16, R55.1
- new net: J1.B2, R62.1
- new net: J1.B4, P20.1 (Pin_1)
- new net: J1.B5, R61.1
- new net: J1.B6, P21.1 (Pin_1)
- new net: J1.B9, R60.1
- new net: J1.C11, P29.1 (Pin_1)
- new net: J1.C12, P30.1 (Pin_1)
- new net: J1.C8, P26.1 (Pin_1)
- new net: J1.C9, P27.1 (Pin_1)
- new net: J1.D1, P31.1 (Pin_1)
- new net: J1.D10, P37.1 (Pin_1)
- new net: J1.D11, R51.1
- new net: J1.D14, R48.1
- new net: J1.D17, R46.1
- new net: J1.D18, R45.1
- new net: J1.D3, R53.1
- new net: J1.D4, R52.1
- new net: J1.D5, P32.1 (Pin_1)
- new net: J1.D6, P33.1 (Pin_1)
- new net: J1.D9, P36.1 (Pin_1)
- new net: U12.1 (OUT), U12.5 (OUT)
- no-connect marks 30 -> 32
Other:
- note added: "TCM MAP TPS"
- note removed: "A"
- note removed: "B"
- note removed: "C"
- note removed: "D"
- note removed: "E"
- moved on the sheet: BT1, C33, D1, F1, F2, F3, F4, H1, H2, H3, H4, J6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
